File: esteemo_hardware/esteemo.kicad_pcb (KiCad board)
At the start: 2 copper layers, 62.4 x 38.1 mm, 30 parts, among them J1 USB_B_Micro, J2 I2S_PMOD_CON, J3 SPI_PMOD_CON, J4 I2C_PMOD_CON, J5 UART_PMOD_CON, J6 SWD_DEBUG_CON, U1 AMS1117-3.3, U2 STM32G0B0CxTx, U3 USBLC6-2SC6, Y1 24MHz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

Commit message: Review PCB and prepare ordering
Parts:
- added D3: DIODE, Diode_SMD:D_SOD-323, F.Cu at (118.4, 93.0)
- C1, C2, C3, C4: value 22n -> 22p
- C5, C6: footprint Capacitor_Tantalum_SMD:CP_EIA-6032-15_Kemet-U -> Capacitor_Tantalum_SMD:CP_EIA-3216-18_Kemet-A
- D2: footprint Diode_SMD:D_0805_2012Metric -> Diode_SMD:D_SOD-323
- FB1: footprint Resistor_SMD:R_1206_3216Metric -> Resistor_SMD:R_0805_2012Metric
- J6: footprint Connector_PinHeader_2.54mm:PinHeader_1x04_P2.54mm_Vertical -> Connector_PinHeader_1.27mm:PinHeader_2x05_P1.27mm_Vertical
- R1: value 4k7 -> 1k
- U1: footprint Package_TO_SOT_SMD:SOT-223-3_TabPin2 -> Package_TO_SOT_SMD:SOT-223
- U3: value USBLC6-2SC6 -> USBLC6-2
- Y1: value 24MHz -> Crystal_GND24; footprint Crystal:Crystal_SMD_G8-2Pin_3.2x1.5mm_HandSoldering -> Crystal:Crystal_SMD_2016-4Pin_2.0x1.6mm
- Y2: footprint Crystal:Crystal_SMD_G8-2Pin_3.2x1.5mm_HandSoldering -> Crystal:Crystal_SMD_3215-2Pin_3.2x1.5mm
- moved R1 9.80 mm to (124.3, 96.3)
- moved D1 9.15 mm to (121.9, 94.0), turned to 180 degrees
- moved J6 6.20 mm to (166.8, 94.0), turned to 0 degrees
- moved C2 4.34 mm to (148.8, 99.6), turned to 90 degrees
- moved C1 2.52 mm to (151.1, 94.2)
- moved FB1 2.34 mm to (121.4, 91.7)
- moved C8 1.83 mm to (121.2, 87.4)
- moved C6 1.78 mm to (136.7, 87.6)
- moved C5 1.48 mm to (120.7, 89.7)
- moved Y1 0.81 mm to (149.4, 96.5), turned to 180 degrees
- turned Y2 to 90 degrees
Connections:
- D1 pad 2: VBUS -> Net-(D1-Pad2)
- FB1 pad 1: VBUS -> Net-(D1-Pad2)
- J6 pad 1: /SWDIO -> +3.3V
- J6 pad 2: /SWCLK -> /SWDIO
- J6 pad 4: +3.3V -> /SWCLK
- Y1 pad 2: /OSC_IN -> GND
Routing:
- net /SWDIO: track 53.5 -> 63.5 mm
- net VBUS: track 16.3 -> 10.7 mm
- net /SWCLK: track 52.6 -> 57.1 mm
- net Net-(D1-Pad2): track 0.00 -> 4.52 mm
- net Net-(C5-Pad1): track 15.0 -> 10.9 mm
- net GND: track 24.2 -> 20.7 mm, vias 14 -> 16
- net +3.3V: track 192.9 -> 190.1 mm
- net /OSC_IN: track 13.6 -> 10.8 mm
- net Net-(D1-Pad1): track 2.60 -> 2.06 mm
Other:
- board text added: "Esteemo v1 07/2022"
