File: esteemo_hardware/esteemo.kicad_sch (KiCad schematic)
At the start: 30 parts, among them J1 USB_B_Micro, J2 I2S_PMOD_CON, J3 SPI_PMOD_CON, J4 I2C_PMOD_CON, J5 UART_PMOD_CON, J6 SWD_DEBUG_CON, U1 AMS1117-3.3, U2 STM32G0B0CxTx, U3 USBLC6-2SC6, Y1 24MHz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

Commit message: Review PCB and prepare ordering
Parts:
- removed J6: SWD_DEBUG_CON, Connector_PinHeader_2.54mm:PinHeader_1x04_P2.54mm_Vertical, symbol Connector:Conn_01x04_Male
- removed Y1: 24MHz, Crystal:Crystal_SMD_G8-2Pin_3.2x1.5mm_HandSoldering, symbol Device:Crystal
- added D3: DIODE, Diode_SMD:D_SOD-323, symbol pspice:DIODE
- added J6: SWD_DEBUG_CON, Connector_PinHeader_1.27mm:PinHeader_2x05_P1.27mm_Vertical, symbol Connector_Generic:Conn_02x05_Odd_Even
- added Y1: Crystal_GND24, Crystal:Crystal_SMD_2016-4Pin_2.0x1.6mm, symbol Device:Crystal_GND24
- C1, C2, C3, C4: value 22n -> 22p; Comment (none) -> https://jlcpcb.com/partdetail/2156-CL21C220JBANNNC/C1804; LCSC_MPN (none) -> C1804
- C10, C7, C8: Comment (none) -> https://jlcpcb.com/partdetail/Avx-TAJA104K035RNJ/C7173; LCSC_MPN (none) -> C7173
- C5, C6: footprint Capacitor_Tantalum_SMD:CP_EIA-6032-15_Kemet-U -> Capacitor_Tantalum_SMD:CP_EIA-3216-18_Kemet-A; Comment (none) -> https://jlcpcb.com/parts/componentSearch?isSecondLevel=true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; LCSC_MPN (none) -> C7171
- D1: Comment (none) -> https://jlcpcb.com/partdetail/EverlightElec-15_21_R6C_FQ1R1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; LCSC_MPN (none) -> C93133
- D2: footprint Diode_SMD:D_0805_2012Metric -> Diode_SMD:D_SOD-323; Comment (none) -> https://jlcpcb.com/partdetail/Toshiba-CUS10S30H3F/C146335; LCSC_MPN (none) -> C146335
- FB1: footprint Resistor_SMD:R_1206_3216Metric -> Resistor_SMD:R_0805_2012Metric; Comment (none) -> https://jlcpcb.com/parts/componentSearch?isSecondLevel=true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; LCSC_MPN (none) -> C1017
- H1, H2, H3, H4: Comment (none) -> Drilled holes; now left out of the parts list
- J1: Comment (none) -> https://jlcpcb.com/partdetail/AmphenolIcc-101181940001LF/C1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; LCSC_MPN (none) -> C132563
- J2, J3, J4, J5: Comment (none) -> https://jlcpcb.com/partdetail/XkbConnectivity-X6511FV_06C85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; LCSC_MPN (none) -> C718239
- R1: value 4k7 -> 1k; Comment (none) -> https://jlcpcb.com/partdetail/18201-0805W8F1001T5E/C17513; LCSC_MPN (none) -> C17513
- R2, R3: Comment (none) -> https://jlcpcb.com/partdetail/18201-0805W8F1001T5E/C17513; LCSC_MPN (none) -> C17513
- U1: footprint Package_TO_SOT_SMD:SOT-223-3_TabPin2 -> Package_TO_SOT_SMD:SOT-223; Comment (none) -> https://jlcpcb.com/partdetail/Advanced_MonolithicSystems-AM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; LCSC_MPN (none) -> C6186
- U2: Comment (none) -> https://jlcpcb.com/partdetail/Stmicroelectronics-STM32G030C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; LCSC_MPN (none) -> C529329
- U3: value USBLC6-2SC6 -> USBLC6-2; Comment (none) -> https://jlcpcb.com/partdetail/Stmicroelectronics-USBLC62SC6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; LCSC_MPN (none) -> C7519
- Y2: footprint Crystal:Crystal_SMD_G8-2Pin_3.2x1.5mm_HandSoldering -> Crystal:Crystal_SMD_3215-2Pin_3.2x1.5mm; Comment (none) -> https://jlcpcb.com/partdetail/SeikoEpson-Q13FC1350000400/C3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; LCSC_MPN (none) -> C32346
Connections:
- net +3.3V: now also J6.1 (Pin_1)
- net GND: now also J6.3 (Pin_3), J6.5 (Pin_5), J6.9 (Pin_9), Y1.2, Y1.4
- net OSC_IN: now also Y1.3
- net OSC_OUT: now also Y1.1
- net SWCLK: now also J6.4 (Pin_4)
- net SWDIO: now also J6.2 (Pin_2)
- net VBUS: now also D3.1 (K); no longer D1.2 (A), FB1.1
- new net: D1.2 (A), D3.2 (A), FB1.1
- no-connect marks 29 -> 33
Other:
- note added: "ARM 10 pin SWD connector"
- moved on the sheet: C5, C6, C8, D1, D2, FB1, R1, U1
